Commit message: rename model.urdf to modelForWalking.urdf

File: app/robots/iCubGenova02/modelForWalking.urdf (robot description, URDF)
Before this commit: robot iCub, 140 links, 139 joints
Links:
- removed link root_link_imu_frame
- link chest: geometry collision mesh filename=package://iCub/meshes/simmechanics/sim_sea_2-5_chest_bb_prt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 scale=0.001 0.001 0.001; visual mesh filename=package://iCub/meshes/simmechanics/sim_sea_2-5_chest_bb_prt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 scale=0.001 0.001 0.001
- link head: geometry collision mesh filename=package://iCub/meshes/simmechanics/sim_sea_2-5_head_prt-bin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 scale=0.001 0.001 0.001; visual mesh filename=package://iCub/meshes/simmechanics/sim_sea_2-5_head_prt-bin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 scale=0.001 0.001 0.001
- link l_ankle_1: geometry collision mesh filename=package://iCub/meshes/simmechanics/sim_sea_2-5_l_ankle_prt-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 scale=0.001 0.001 0.001; visual mesh filename=package://iCub/meshes/simmechanics/sim_sea_2-5_l_ankle_prt-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 scale=0.001 0.001 0.001
- link l_ankle_2: mass 0.265337 -> 0.267485; geometry collision mesh filename=package://iCub/meshes/simmechanics/sim_sea_2-5_l_foot_prt-b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 scale=0.001 0.001 0.001; visual mesh filename=package://iCub/meshes/simmechanics/sim_sea_2-5_l_foot_prt-b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 scale=0.001 0.001 0.001
- link l_elbow_1: geometry collision mesh filename=package://iCub/meshes/simmechanics/sim_sea_2-5_l_elbow_pros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 scale=0.001 0.001 0.001; visual mesh filename=package://iCub/meshes/simmechanics/sim_sea_2-5_l_elbow_pros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 scale=0.001 0.001 0.001
- link l_foot: mass 0.357881 -> 0.382968; geometry collision mesh filename=package://iCub/meshes/simmechanics/sim_sea_2-5_l_sole_prt-b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 scale=0.001 0.001 0.001; visual mesh filename=package://iCub/meshes/simmechanics/sim_sea_2-5_l_sole_prt-b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 scale=0.001 0.001 0.001
- link l_forearm: geometry collision mesh filename=package://iCub/meshes/simmechanics/sim_sea_2-5_l_forearm_pr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 scale=0.001 0.001 0.001; visual mesh filename=package://iCub/meshes/simmechanics/sim_sea_2-5_l_forearm_pr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 scale=0.001 0.001 0.001
- link l_hand: geometry collision mesh filename=package://iCub/meshes/simmechanics/sim_sea_2-5_l_hand_prt-b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 scale=0.001 0.001 0.001; visual mesh filename=package://iCub/meshes/simmechanics/sim_sea_2-5_l_hand_prt-b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 scale=0.001 0.001 0.001
- link l_hip_1: geometry collision mesh filename=package://iCub/meshes/simmechanics/sim_sea_2-5_l_hip_1_prt-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 scale=0.001 0.001 0.001; visual mesh filename=package://iCub/meshes/simmechanics/sim_sea_2-5_l_hip_1_prt-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 scale=0.001 0.001 0.001
- link l_hip_2: geometry collision mesh filename=package://iCub/meshes/simmechanics/sim_sea_2-5_l_hip_2_prt-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 scale=0.001 0.001 0.001; visual mesh filename=package://iCub/meshes/simmechanics/sim_sea_2-5_l_hip_2_prt-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 scale=0.001 0.001 0.001
- link l_hip_3: geometry collision mesh filename=package://iCub/meshes/simmechanics/sim_sea_2-5_l_upper_thig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 scale=0.001 0.001 0.001; visual mesh filename=package://iCub/meshes/simmechanics/sim_sea_2-5_l_upper_thig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 scale=0.001 0.001 0.001
- link l_lower_leg: geometry collision mesh filename=package://iCub/meshes/simmechanics/sim_sea_2-5_l_shank_prt-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 scale=0.001 0.001 0.001; visual mesh filename=package://iCub/meshes/simmechanics/sim_sea_2-5_l_shank_prt-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 scale=0.001 0.001 0.001
- link l_shoulder_1: geometry collision mesh filename=package://iCub/meshes/simmechanics/sim_sea_2-5_l_shoulder_1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 scale=0.001 0.001 0.001; visual mesh filename=package://iCub/meshes/simmechanics/sim_sea_2-5_l_shoulder_1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 scale=0.001 0.001 0.001
- link l_shoulder_2: geometry collision mesh filename=package://iCub/meshes/simmechanics/sim_sea_2-5_l_shoulder_2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 scale=0.001 0.001 0.001; visual mesh filename=package://iCub/meshes/simmechanics/sim_sea_2-5_l_shoulder_2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 scale=0.001 0.001 0.001
- link l_shoulder_3: geometry collision mesh filename=package://iCub/meshes/simmechanics/sim_sea_2-5_l_upper_arm_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 scale=0.001 0.001 0.001; visual mesh filename=package://iCub/meshes/simmechanics/sim_sea_2-5_l_upper_arm_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 scale=0.001 0.001 0.001
- link l_upper_arm: geometry collision mesh filename=package://iCub/meshes/simmechanics/sim_sea_2-5_l_elbow_prt-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 scale=0.001 0.001 0.001; visual mesh filename=package://iCub/meshes/simmechanics/sim_sea_2-5_l_elbow_prt-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 scale=0.001 0.001 0.001
- link l_upper_leg: geometry collision mesh filename=package://iCub/meshes/simmechanics/sim_sea_2-5_l_thigh_prt-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 scale=0.001 0.001 0.001; visual mesh filename=package://iCub/meshes/simmechanics/sim_sea_2-5_l_thigh_prt-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 scale=0.001 0.001 0.001
- link l_wrist_1: geometry collision mesh filename=package://iCub/meshes/simmechanics/sim_sea_2-5_l_wrist_pitc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 scale=0.001 0.001 0.001; visual mesh filename=package://iCub/meshes/simmechanics/sim_sea_2-5_l_wrist_pitc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 scale=0.001 0.001 0.001
- link neck_1: geometry collision mesh filename=package://iCub/meshes/simmechanics/sim_sea_2-5_neck_1_prt-b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 scale=0.001 0.001 0.001; visual mesh filename=package://iCub/meshes/simmechanics/sim_sea_2-5_neck_1_prt-b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 scale=0.001 0.001 0.001
- link neck_2: geometry collision mesh filename=package://iCub/meshes/simmechanics/sim_sea_2-5_neck_2_prt-b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 scale=0.001 0.001 0.001; visual mesh filename=package://iCub/meshes/simmechanics/sim_sea_2-5_neck_2_prt-b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 scale=0.001 0.001 0.001
- link r_ankle_1: geometry collision mesh filename=package://iCub/meshes/simmechanics/sim_sea_2-5_r_ankle_prt-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 scale=0.001 0.001 0.001; visual mesh filename=package://iCub/meshes/simmechanics/sim_sea_2-5_r_ankle_prt-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 scale=0.001 0.001 0.001
- link r_ankle_2: mass 0.265337 -> 0.267485; geometry collision mesh filename=package://iCub/meshes/simmechanics/sim_sea_2-5_r_foot_prt-b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 scale=0.001 0.001 0.001; visual mesh filename=package://iCub/meshes/simmechanics/sim_sea_2-5_r_foot_prt-b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 scale=0.001 0.001 0.001
- link r_elbow_1: geometry collision mesh filename=package://iCub/meshes/simmechanics/sim_sea_2-5_r_elbow_pros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 scale=0.001 0.001 0.001; visual mesh filename=package://iCub/meshes/simmechanics/sim_sea_2-5_r_elbow_pros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 scale=0.001 0.001 0.001
- link r_foot: mass 0.357881 -> 0.382866; geometry collision mesh filename=package://iCub/meshes/simmechanics/sim_sea_2-5_r_sole_prt-b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 scale=0.001 0.001 0.001; visual mesh filename=package://iCub/meshes/simmechanics/sim_sea_2-5_r_sole_prt-b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 scale=0.001 0.001 0.001
- link r_forearm: geometry collision mesh filename=package://iCub/meshes/simmechanics/sim_sea_2-5_r_forearm_pr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 scale=0.001 0.001 0.001; visual mesh filename=package://iCub/meshes/simmechanics/sim_sea_2-5_r_forearm_pr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 scale=0.001 0.001 0.001
- link r_hand: geometry collision mesh filename=package://iCub/meshes/simmechanics/sim_sea_2-5_r_hand_prt-b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 scale=0.001 0.001 0.001; visual mesh filename=package://iCub/meshes/simmechanics/sim_sea_2-5_r_hand_prt-b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 scale=0.001 0.001 0.001
- link r_hip_1: geometry collision mesh filename=package://iCub/meshes/simmechanics/sim_sea_2-5_r_hip_1_prt-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 scale=0.001 0.001 0.001; visual mesh filename=package://iCub/meshes/simmechanics/sim_sea_2-5_r_hip_1_prt-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 scale=0.001 0.001 0.001
- link r_hip_2: geometry collision mesh filename=package://iCub/meshes/simmechanics/sim_sea_2-5_r_hip_2_prt-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 scale=0.001 0.001 0.001; visual mesh filename=package://iCub/meshes/simmechanics/sim_sea_2-5_r_hip_2_prt-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 scale=0.001 0.001 0.001
- link r_hip_3: geometry collision mesh filename=package://iCub/meshes/simmechanics/sim_sea_2-5_r_upper_thig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 scale=0.001 0.001 0.001; visual mesh filename=package://iCub/meshes/simmechanics/sim_sea_2-5_r_upper_thig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 scale=0.001 0.001 0.001
- link r_lower_leg: geometry collision mesh filename=package://iCub/meshes/simmechanics/sim_sea_2-5_r_shank_prt-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 scale=0.001 0.001 0.001; visual mesh filename=package://iCub/meshes/simmechanics/sim_sea_2-5_r_shank_prt-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 scale=0.001 0.001 0.001
- link r_shoulder_1: geometry collision mesh filename=package://iCub/meshes/simmechanics/sim_sea_2-5_r_shoulder_1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 scale=0.001 0.001 0.001; visual mesh filename=package://iCub/meshes/simmechanics/sim_sea_2-5_r_shoulder_1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 scale=0.001 0.001 0.001
- link r_shoulder_2: geometry collision mesh filename=package://iCub/meshes/simmechanics/sim_sea_2-5_r_shoulder_2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 scale=0.001 0.001 0.001; visual mesh filename=package://iCub/meshes/simmechanics/sim_sea_2-5_r_shoulder_2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 scale=0.001 0.001 0.001
- link r_shoulder_3: geometry collision mesh filename=package://iCub/meshes/simmechanics/sim_sea_2-5_r_upper_arm_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 scale=0.001 0.001 0.001; visual mesh filename=package://iCub/meshes/simmechanics/sim_sea_2-5_r_upper_arm_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 scale=0.001 0.001 0.001
- link r_upper_arm: geometry collision mesh filename=package://iCub/meshes/simmechanics/sim_sea_2-5_r_elbow_prt-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 scale=0.001 0.001 0.001; visual mesh filename=package://iCub/meshes/simmechanics/sim_sea_2-5_r_elbow_prt-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 scale=0.001 0.001 0.001
- link r_upper_leg: geometry collision mesh filename=package://iCub/meshes/simmechanics/sim_sea_2-5_r_thigh_prt-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 scale=0.001 0.001 0.001; visual mesh filename=package://iCub/meshes/simmechanics/sim_sea_2-5_r_thigh_prt-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 scale=0.001 0.001 0.001
- link r_wrist_1: geometry collision mesh filename=package://iCub/meshes/simmechanics/sim_sea_2-5_r_wrist_pitc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 scale=0.001 0.001 0.001; visual mesh filename=package://iCub/meshes/simmechanics/sim_sea_2-5_r_wrist_pitc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 scale=0.001 0.001 0.001
- link root_link: mass 5.12739 -> 5.09143; geometry collision mesh filename=package://iCub/meshes/simmechanics/sim_sea_2-5_root_link_pr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 scale=0.001 0.001 0.001; visual mesh filename=package://iCub/meshes/simmechanics/sim_sea_2-5_root_link_pr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 scale=0.001 0.001 0.001
- link torso_1: geometry collision mesh filename=package://iCub/meshes/simmechanics/sim_sea_2-5_lap_belt_1_p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 scale=0.001 0.001 0.001; visual mesh filename=package://iCub/meshes/simmechanics/sim_sea_2-5_lap_belt_1_p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 scale=0.001 0.001 0.001
- link torso_2: geometry collision mesh filename=package://iCub/meshes/simmechanics/sim_sea_2-5_lap_belt_2_p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 scale=0.001 0.001 0.001; visual mesh filename=package://iCub/meshes/simmechanics/sim_sea_2-5_lap_belt_2_p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 scale=0.001 0.001 0.001
Joints:
- removed joint root_link_imu_frame_fixed_joint
- joint l_ankle_pitch: axis -6.66133814775e-16 1.0 4.4408920985e-16 -> 2.22044604925e-16 1.0 0.0; limit lower=-0.872664625997 upper=0.349065850399 effort=37.0 velocity=7.64 -> lower=-0.610865238198 upper=0.610865238198 effort=37.0 velocity=7.64; origin xyz=0 0 -0.2005 rpy=0 0.26179917948 0 -> xyz=0 0 -0.2005 rpy=0 0 0
- joint l_ankle_roll: axis 1.00000015612 6.0136540192e-16 -1.19793949732e-07 -> 1.0 0.0 2.22044604925e-16
- joint l_foot_ft_sensor: origin xyz=-0.00349992806597 0 -0.0605003432802 rpy=-3.14159264324 0 0 -> xyz=-0.0035 0 -0.0605 rpy=3.14159265359 0 0
- joint l_hip_yaw: origin xyz=0 0 0.0144 rpy=-3.14159265359 0 0 -> xyz=0 0 0.0144 rpy=-3.14159265359 0 -1.57079632679
- joint l_knee: axis -2.22044604925e-16 -1.0 0.0 -> -2.22044604925e-16 -1.0 -0.0
- joint l_leg_ft_sensor: origin xyz=-0.0008575 0 -0.0743 rpy=3.14159265359 0 0 -> xyz=-0.0008575 0 -0.0743 rpy=-3.14159265359 0 -1.57079632679
- joint l_sole_fixed_joint: origin xyz=0.0214502260596 0 0.00669127665248 rpy=-3.14159265359 0.261799192098 0 -> xyz=0.0035 0 0.004 rpy=-3.14159265359 0 0
- joint r_ankle_pitch: axis -6.66133814775e-16 1.0 4.4408920985e-16 -> 2.22044604925e-16 1.0 0.0; limit lower=-0.872664625997 upper=0.349065850399 effort=37.0 velocity=7.64 -> lower=-0.610865238198 upper=0.610865238198 effort=37.0 velocity=7.64; origin xyz=0 0 -0.2005 rpy=0 0.26179917948 0 -> xyz=0 0 -0.2005 rpy=0 0 0
- joint r_ankle_roll: axis -1.00000015612 -6.0136540192e-16 1.19793949732e-07 -> -1.0 -0.0 -2.22044604925e-16
- joint r_foot_ft_sensor: origin xyz=-0.00349992806597 0 -0.0605003432802 rpy=3.14159265242 0 0 -> xyz=-0.0035 0 -0.0605 rpy=3.14159265359 0 0
- joint r_hip_pitch: axis -2.22044604925e-16 -1.0 0.0 -> -2.22044604925e-16 -1.0 -0.0
- joint r_sole_fixed_joint: origin xyz=0.0214502260596 0 0.00669127665248 rpy=-3.14159265359 0.261799181028 0 -> xyz=0.0035 0 0.004 rpy=-3.14159265359 0 0
- joint torso_pitch: origin xyz=0 0.0269348 0 rpy=1.57079632679 0 -1.57079632679 -> xyz=0 0.0270463 0 rpy=1.57079632679 0 -1.57079632679
- joint torso_roll: origin xyz=0.0269347998093 0.032 -0.0573446 rpy=0 0 0 -> xyz=0.0270462998093 0.032 -0.0573446 rpy=0 0 0
